Commit message: sim: maze world (map+nav), ground-truth exporter, camera + IMU noise in robot model, world features spawner
Co-Authored-By: Claude Sonnet 5.5 <noreply@anthropic.com>
Claude-Session: https://claude.ai/code/session_01TwjVqtwKjhx7wg3khDuKdH

File: ros2_ws/src/rdj2026_sim/urdf/hardleel_sim.urdf (robot description, URDF)
Before this commit: robot hardleel, 7 links, 6 joints
Links:
- added link camera, mass 0.01; visual box size=0.02 0.05 0.03
Joints:
- added joint camera_joint: type fixed, parent base_link, child camera, origin xyz=0.10 0 0.20 rpy=0 0 0

Commit message: sim: 4-wheel skid-steer model, ramps/features, SIM_REPORT, blockers, regression scripts
Co-Authored-By: Claude Sonnet 5.5 <noreply@anthropic.com>
Claude-Session: https://claude.ai/code/session_01TwjVqtwKjhx7wg3khDuKdH

File: ros2_ws/src/rdj2026_sim/urdf/hardleel_sim.urdf (robot description, URDF)
Before this commit: robot hardleel, 8 links, 7 joints
Links:
- removed link caster_back
- removed link caster_front
- removed link left_wheel
- removed link right_wheel
- added link front_left_wheel, mass 0.08; collision cylinder length=0.025 radius=0.035; visual cylinder length=0.025 radius=0.035
- added link front_right_wheel, mass 0.08; collision cylinder length=0.025 radius=0.035; visual cylinder length=0.025 radius=0.035
- added link rear_left_wheel, mass 0.08; collision cylinder length=0.025 radius=0.035; visual cylinder length=0.025 radius=0.035
- added link rear_right_wheel, mass 0.08; collision cylinder length=0.025 radius=0.035; visual cylinder length=0.025 radius=0.035
Joints:
- removed joint caster_back_joint
- removed joint caster_front_joint
- removed joint left_wheel_joint
- removed joint right_wheel_joint
- added joint front_left_wheel_joint: type continuous, parent base_link, child front_left_wheel, origin xyz=0.10 0.1225 0, axis 0 1 0
- added joint front_right_wheel_joint: type continuous, parent base_link, child front_right_wheel, origin xyz=0.10 -0.1225 0, axis 0 1 0
- added joint rear_left_wheel_joint: type continuous, parent base_link, child rear_left_wheel, origin xyz=-0.10 0.1225 0, axis 0 1 0
- added joint rear_right_wheel_joint: type continuous, parent base_link, child rear_right_wheel, origin xyz=-0.10 -0.1225 0, axis 0 1 0
